File: hw/DykoDAC3_DAC.kicad_sch (KiCad schematic)
At the start: 56 parts

Commit message: ...
Parts:
- C? (x6): value 100n -> 1u
Changed lines of the file:
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@@
-(kicad_sch (version 20210126) (generator eeschema)
+(kicad_sch (version 20210621) (generator eeschema)
   (paper "A4")
   (junction (at 45.72 40.005) (diameter 1.016) (color 0 0 0 0))
@@
     (in_bom yes) (on_board yes)
     (property "Reference" "C?" (id 0) (at 57.785 113.03 90))
-    (property "Value" "100n" (id 1) (at 58.42 115.57 90))
+    (property "Value" "1u" (id 1) (at 58.42 115.57 90))
     (property "Footprint" "" (id 2) (at 62.23 114.3 0)
       (effects (font (size 1.27 1.27)) hide)
@@
     (in_bom yes) (on_board yes)
     (property "Reference" "C?" (id 0) (at 81.915 113.03 90))
-    (property "Value" "100n" (id 1) (at 83.185 115.57 90))
+    (property "Value" "1u" (id 1) (at 83.185 115.57 90))
     (property "Footprint" "" (id 2) (at 80.01 114.3 0)
       (effects (font (size 1.27 1.27)) hide)
@@
     (in_bom yes) (on_board yes)
     (property "Reference" "C?" (id 0) (at 163.195 91.44 90))
-    (property "Value" "100n" (id 1) (at 162.56 94.615 90))
+    (property "Value" "1u" (id 1) (at 162.56 94.615 90))
     (property "Footprint" "" (id 2) (at 165.735 93.345 0)
       (effects (font (size 1.27 1.27)) hide)
@@
     (in_bom yes) (on_board yes)
     (property "Reference" "C?" (id 0) (at 194.945 91.44 90))
-    (property "Value" "100n" (id 1) (at 195.58 94.615 90))
+    (property "Value" "1u" (id 1) (at 195.58 94.615 90))
     (property "Footprint" "" (id 2) (at 192.405 93.345 0)
       (effects (font (size 1.27 1.27)) hide)
@@
     (in_bom yes) (on_board yes)
     (property "Reference" "C?" (id 0) (at 236.22 92.075 90))
-    (property "Value" "100n" (id 1) (at 235.585 95.25 90))
+    (property "Value" "1u" (id 1) (at 235.585 95.25 90))
     (property "Footprint" "" (id 2) (at 238.76 93.98 0)
       (effects (font (size 1.27 1.27)) hide)
@@
     (in_bom yes) (on_board yes)
     (property "Reference" "C?" (id 0) (at 267.97 92.075 90))
-    (property "Value" "100n" (id 1) (at 268.605 95.25 90))
+    (property "Value" "1u" (id 1) (at 268.605 95.25 90))
     (property "Footprint" "" (id 2) (at 265.43 93.98 0)
       (effects (font (size 1.27 1.27)) hide)

Commit message: no message
Connections:
- net DAC_VREF renamed DAC_VREF_2390mV
Other:
- moved on the sheet: C?, D?, Q?A, Q?B, R?
