File: hw/DykoDAC3_MCUPower.kicad_sch (KiCad schematic)
At the start: 34 parts

Commit message: ...
Parts:
- added C?: 1u, symbol Device:C_Small
- added U?: IMXRT1010, symbol imx:IMXRT1010
- added U?: AT25SF081-SSHD-X, Package_SO:SOIC-8_3.9x4.9mm_P1.27mm, symbol Memory_Flash:AT25SF081-SSHD-X
Connections:
- net GNDD: now also C?.2, U?.4 (GND), U?.72 (GPIO_SD_04/BOOT0), U?.73 (GPIO_SD_03/BOOT1), U?.74 (GPIO_SD_02), U?.75 (GPIO_SD_01), U?.76 (GPIO_SD_00)
- net VCC: now also C?.1, U?.8 (VCC)
- new net FLASH_CS: U?.1 (~{CS}), U?.69 (GPIO_SD_06/QSPI_CS)
- new net FLASH_IO0: U?.5 (SI/IO0), U?.66 (GPIO_SD_09/QSPI_IO0)
- new net FLASH_IO1: U?.2 (SO/IO1), U?.68 (GPIO_SD_07/QSPI_IO1)
- new net FLASH_IO2: U?.3 (~{WP}/IO2), U?.67 (GPIO_SD_08/QSPI_IO2)
- new net FLASH_IO3: U?.64 (GPIO_SD_11/QSPI_IO3), U?.7 (~{HOLD}/IO3)
- new net FLASH_SCK: U?.6 (SCK), U?.65 (GPIO_SD_10/QSPI_SCK)
- no-connect marks 5 -> 8
Other:
- moved on the sheet: C?, R?, U?B, U?C, Y?

Commit message: no message
Parts:
- added R?: 10k, symbol Device:R_Small
- added U? (x2): IMXRT1010, symbol imx:IMXRT1010
Connections:
- net FLASH_CS: now also R?.1
- net VCC: now also R?.2
- new net DCDC_EN: U?.57 (GPIO_AD_03)
Other:
- moved on the sheet: C?, U?, U?C, U?F
