File: hw/DykoDAC3_Power.kicad_sch (KiCad schematic)
At the start: 26 parts

Commit message: imx power
Connections:
- net USDB_D- renamed USB_D-
Changed lines of the file:
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@@
-    (stroke (width 0) (type solid) (color 0 0 0 0))
-  )
-  (wire (pts (xy 49.53 25.4) (xy 63.5 25.4))
     (stroke (width 0) (type solid) (color 0 0 0 0))
   )
@@
     (stroke (width 0) (type solid) (color 0 0 0 0))
   )
+  (wire (pts (xy 62.23 25.4) (xy 49.53 25.4))
+    (stroke (width 0) (type solid) (color 0 0 0 0))
+  )
   (wire (pts (xy 62.23 27.94) (xy 53.34 27.94))
     (stroke (width 0) (type solid) (color 0 0 0 0))
@@
     (stroke (width 0) (type solid) (color 0 0 0 0))
   )
-  (global_label "USDB_D-" (shape input) (at 62.23 27.94 0) (fields_autoplaced)
+  (global_label "USB_D+" (shape input) (at 62.23 25.4 0) (fields_autoplaced)
     (effects (font (size 1.27 1.27)) (justify left))
-    (property "Intersheet References" "${INTERSHEET_REFS}" (id 0) (at 0 0 0)
+    (property "Intersheet References" "${INTERSHEET_REFS}" (id 0) (at -1.27 0 0)
       (effects (font (size 1.27 1.27)) hide)
     )
   )
-  (global_label "USB_D+" (shape input) (at 63.5 25.4 0) (fields_autoplaced)
+  (global_label "USB_D-" (shape input) (at 62.23 27.94 0) (fields_autoplaced)
     (effects (font (size 1.27 1.27)) (justify left))
-    (property "Intersheet References" "${INTERSHEET_REFS}" (id 0) (at 0 0 0)
-      (effects (font (size 1.27 1.27)) hide)
+    (property "Intersheet References" "${INTERSHEET_REFS}" (id 0) (at 72.2631 27.8606 0)
+      (effects (font (size 1.27 1.27)) (justify left) hide)
     )
   )

Commit message: ...
Parts:
- removed C?: 1n, symbol DykoDAC3-rescue:C_Small-Device
- removed R?: 1M, symbol DykoDAC3-rescue:R_Small-Device
- C?: value 100n -> 1u
Connections:
- no-connect marks 0 -> 1
Changed lines of the file:
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@@
-(kicad_sch (version 20210126) (generator eeschema)
+(kicad_sch (version 20210621) (generator eeschema)
   (paper "A4")
-  (junction (at 25.4 40.64) (diameter 1.016) (color 0 0 0 0))
-  (junction (at 25.4 49.53) (diameter 1.016) (color 0 0 0 0))
-  (junction (at 31.75 38.1) (diameter 1.016) (color 0 0 0 0))
-  (junction (at 39.37 20.32) (diameter 1.016) (color 0 0 0 0))
+  (junction (at 27.94 38.1) (diameter 1.016) (color 0 0 0 0))
   (junction (at 49.53 25.4) (diameter 1.016) (color 0 0 0 0))
   (junction (at 53.34 27.94) (diameter 1.016) (color 0 0 0 0))
+  (junction (at 57.15 20.32) (diameter 1.016) (color 0 0 0 0))
   (junction (at 85.725 26.035) (diameter 1.016) (color 0 0 0 0))
   (junction (at 85.725 38.735) (diameter 1.016) (color 0 0 0 0))
@@
   (junction (at 250.825 39.37) (diameter 1.016) (color 0 0 0 0))
   (junction (at 250.825 50.8) (diameter 1.016) (color 0 0 0 0))
-  (wire (pts (xy 21.59 40.64) (xy 21.59 41.91))
-    (stroke (width 0) (type solid) (color 0 0 0 0))
-  )
-  (wire (pts (xy 21.59 49.53) (xy 21.59 46.99))
-    (stroke (width 0) (type solid) (color 0 0 0 0))
-  )
-  (wire (pts (xy 25.4 35.56) (xy 25.4 40.64))
-    (stroke (width 0) (type solid) (color 0 0 0 0))
-  )
-  (wire (pts (xy 25.4 40.64) (xy 21.59 40.64))
-    (stroke (width 0) (type solid) (color 0 0 0 0))
-  )
-  (wire (pts (xy 25.4 41.91) (xy 25.4 40.64))
-    (stroke (width 0) (type solid) (color 0 0 0 0))
-  )
-  (wire (pts (xy 25.4 46.99) (xy 25.4 49.53))
-    (stroke (width 0) (type solid) (color 0 0 0 0))
-  )
-  (wire (pts (xy 25.4 49.53) (xy 21.59 49.53))
-    (stroke (width 0) (type solid) (color 0 0 0 0))
-  )
-  (wire (pts (xy 25.4 49.53) (xy 31.75 49.53))
-    (stroke (width 0) (type solid) (color 0 0 0 0))
-  )
-  (wire (pts (xy 25.4 52.07) (xy 25.4 49.53))
-    (stroke (width 0) (type solid) (color 0 0 0 0))
-  )
+  (no_connect (at 25.4 35.56))
   (wire (pts (xy 27.94 35.56) (xy 27.94 38.1))
     (stroke (width 0) (type solid) (color 0 0 0 0))
   )
-  (wire (pts (xy 27.94 38.1) (xy 31.75 38.1))
-    (stroke (width 0) (type solid) (color 0 0 0 0))
-  )
-  (wire (pts (xy 31.75 38.1) (xy 40.64 38.1))
-    (stroke (width 0) (type solid) (color 0 0 0 0))
-  )
-  (wire (pts (xy 31.75 49.53) (xy 31.75 38.1))
+  (wire (pts (xy 27.94 38.1) (xy 40.64 38.1))
+    (stroke (width 0) (type solid) (color 0 0 0 0))
+  )
+  (wire (pts (xy 27.94 40.64) (xy 27.94 38.1))
+    (stroke (width 0) (type solid) (color 0 0 0 0))
+  )
+  (wire (pts (xy 35.56 20.32) (xy 57.15 20.32))
     (stroke (width 0) (type solid) (color 0 0 0 0))
   )
@@
     (stroke (width 0) (type solid) (color 0 0 0 0))
   )
-  (wire (pts (xy 39.37 19.05) (xy 39.37 20.32))
-    (stroke (width 0) (type solid) (color 0 0 0 0))
-  )
-  (wire (pts (xy 39.37 20.32) (xy 35.56 20.32))
-    (stroke (width 0) (type solid) (color 0 0 0 0))
-  )
   (wire (pts (xy 40.64 30.48) (xy 45.72 30.48))
     (stroke (width 0) (type solid) (color 0 0 0 0))
@@
     (stroke (width 0) (type solid) (color 0 0 0 0))
   )
-  (wire (pts (xy 57.15 20.32) (xy 39.37 20.32))
+  (wire (pts (xy 57.15 18.415) (xy 57.15 20.32))
     (stroke (width 0) (type solid) (color 0 0 0 0))
   )
@@
     )
   )
-  (symbol (lib_id "DykoDAC3-rescue:+5V-power") (at 39.37 19.05 0) (unit 1)
-    (in_bom yes) (on_board yes)
-    (property "Reference" "#PWR0106" (id 0) (at 39.37 22.86 0)
-      (effects (font (size 1.27 1.27)) hide)
-    )
-    (property "Value" "+5V" (id 1) (at 39.751 14.6558 0))
-    (property "Footprint" "" (id 2) (at 39.37 19.05 0)
-      (effects (font (size 1.27 1.27)) hide)
-    )
-    (property "Datasheet" "" (id 3) (at 39.37 19.05 0)
+  (symbol (lib_id "DykoDAC3-rescue:+5V-power") (at 57.15 18.415 0) (unit 1)
+    (in_bom yes) (on_board yes)
+    (property "Reference" "#PWR0106" (id 0) (at 57.15 22.225 0)
+      (effects (font (size 1.27 1.27)) hide)
+    )
+    (property "Value" "+5V" (id 1) (at 57.531 14.0208 0))
+    (property "Footprint" "" (id 2) (at 57.15 18.415 0)
+      (effects (font (size 1.27 1.27)) hide)
+    )
+    (property "Datasheet" "" (id 3) (at 57.15 18.415 0)
       (effects (font (size 1.27 1.27)) hide)
     )
@@
     (pin "1")
   )
-  (symbol (lib_id "DykoDAC3-rescue:GNDD-power") (at 25.4 52.07 0) (unit 1)
-    (in_bom yes) (on_board yes)
-    (property "Reference" "#PWR0103" (id 0) (at 25.4 58.42 0)
-      (effects (font (size 1.27 1.27)) hide)
-    )
-    (property "Value" "GNDD" (id 1) (at 25.5016 56.007 0))
-    (property "Footprint" "" (id 2) (at 25.4 52.07 0)
-      (effects (font (size 1.27 1.27)) hide)
-    )
-    (property "Datasheet" "" (id 3) (at 25.4 52.07 0)
+  (symbol (lib_id "DykoDAC3-rescue:GNDD-power") (at 27.94 40.64 0) (unit 1)
+    (in_bom yes) (on_board yes)
+    (property "Reference" "#PWR0103" (id 0) (at 27.94 46.99 0)
+      (effects (font (size 1.27 1.27)) hide)
+    )
+    (property "Value" "GNDD" (id 1) (at 28.0416 44.577 0))
+    (property "Footprint" "" (id 2) (at 27.94 40.64 0)
+      (effects (font (size 1.27 1.27)) hide)
+    )
+    (property "Datasheet" "" (id 3) (at 27.94 40.64 0)
       (effects (font (size 1.27 1.27)) hide)
     )
@@
     (pin "2")
   )
-  (symbol (lib_id "DykoDAC3-rescue:R_Small-Device") (at 25.4 44.45 0) (unit 1)
-    (in_bom yes) (on_board yes)
-    (property "Reference" "R?" (id 0) (at 26.8986 43.2816 0)
-      (effects (font (size 1.27 1.27)) (justify left))
-    )
-    (property "Value" "1M" (id 1) (at 26.8986 45.593 0)
-      (effects (font (size 1.27 1.27)) (justify left))
-    )
-    (property "Footprint" "" (id 2) (at 25.4 44.45 0)
-      (effects (font (size 1.27 1.27)) hide)
-    )
-    (property "Datasheet" "~" (id 3) (at 25.4 44.45 0)
-      (effects (font (size 1.27 1.27)) hide)
-    )
-    (pin "1")
-    (pin "2")
-  )
   (symbol (lib_id "DykoDAC3-rescue:CP_Small-Device") (at 103.505 32.385 0) (unit 1)
     (in_bom yes) (on_board yes)
@@
     )
     (property "Datasheet" "~" (id 3) (at 250.825 44.45 0)
-      (effects (font (size 1.27 1.27)) hide)
-    )
-    (pin "1")
-    (pin "2")
-  )
-  (symbol (lib_id "DykoDAC3-rescue:C_Small-Device") (at 21.59 44.45 0) (unit 1)
-    (in_bom yes) (on_board yes)
-    (property "Reference" "C?" (id 0) (at 16.51 43.18 0)
-      (effects (font (size 1.27 1.27)) (justify left))
-    )
-    (property "Value" "1n" (id 1) (at 16.51 45.72 0)
-      (effects (font (size 1.27 1.27)) (justify left))
-    )
-    (property "Footprint" "" (id 2) (at 21.59 44.45 0)
-      (effects (font (size 1.27 1.27)) hide)
-    )
-    (property "Datasheet" "~" (id 3) (at 21.59 44.45 0)
       (effects (font (size 1.27 1.27)) hide)
     )
@@
     (in_bom yes) (on_board yes)
     (property "Reference" "C?" (id 0) (at 147.32 26.67 90))
-    (property "Value" "100n" (id 1) (at 140.97 26.67 90))
+    (property "Value" "1u" (id 1) (at 141.605 26.67 90))
     (property "Footprint" "" (id 2) (at 144.78 27.94 0)
       (effects (font (size 1.27 1.27)) hide)

Commit message: no message
Parts:
- added C? (x4): 10u, symbol DykoDAC3-rescue:C_Small-Device
- added C?: 47u, symbol DykoDAC3-rescue:C_Small-Device
- added U?: MCP1702T-5, Package_TO_SOT_SMD:SOT-23, symbol Regulator_Linear:MCP1700-1202E_SOT23
- added U?: LP5907MFX-3.3, Package_TO_SOT_SMD:SOT-23-5, symbol Regulator_Linear:LP5907MFX-3.3
- TR?: value DA2304 -> DA2303
Connections:
- net +10V: now also C?.1, U?.3 (VI)
- net +5VD: now also C?.1, C?.1, U?.1 (IN), U?.3 (EN)
- net GNDA: now also C?.2, C?.2, U?.1 (GND)
- net GNDD: now also C?.2, C?.2, C?.2, U?.2 (GND)
- new net VCC: C?.1, U?.5 (OUT)
- new net VCCQ: C?.1, U?.2 (VO)
Other:
- moved on the sheet: C?, D?, L?, TR?, U?
